Commit message: Gazebo: real contact grasp, real control, measured
The Gazebo backend could run an episode and print numbers, but every number was
wrong in a way that only running the physics could reveal. This fixes the eight
defects that were found by measuring the live simulation, and deletes the one
behaviour that was fabricating its result.

Scene and robot (all found by running it)

* world_sdf located the robot with str.replace("<model name='panda'>", ...), but
  robot_model_sdf round-trips the block through xml.etree, which emits
  double-quoted attributes. The replacement never matched, so the robot was
  emitted with NO <pose> at all, spawned at the world origin with its base
  cylinder 20 mm inside the tabletop and ejected by ODE: the panda model was
  measured at z = -10162 m, in free fall, while the arm "moved" and the episode
  reported a grasp. place_robot_model now parses the model, inserts the pose as
  an element, and RAISES if it cannot place it, so a silent no-op cannot recur.
* The arm is now anchored to the world with a fixed joint, which is how a robot
  arm is bolted to a table. joint1's settled error went from 87 mrad -- it was
  fighting the falling base -- to 0.01-0.55 mrad.
* world_sdf drew a 40 mm cube for a 16 mm condition, a table 20% too small, a
  target marker 0.27 m from where the task scores placement, and no friction.
  Object size, mass, inertia, resting height, target zone, table extent, spawn
  annulus and friction are now all derived from the ScenarioConfig.
* The URDF's pads were 50 mm tall boxes 20 mm behind the pad centre and the two
  jaws were asymmetric. Rebuilt from the MJCF measurements: pad centre at
  hand-frame z = 0.1029, half-height 8.5 mm, closed separation 11 mm,
  symmetric by construction, and pinned against RobotConfig by a test.

Frames (the reason the arm never reached anything)

* The IK provider stopped at panda_link7 -- the wrist, 0.2104 m behind the tool
  -- while every waypoint is a tool-centre point. The policy's own "have I
  reached" test could therefore never become true and the waypoint cursor never
  advanced. The chain now runs through the fixed hand_joint to the TCP site at
  hand-frame z = 0.1034, the same frame simulation/mujoco_env.py injects.
* The provider answered in the robot's BASE frame while waypoints, the object
  pose and MuJoCo's provider are all WORLD. Raising the base exposed it: the
  tool settled exactly 20 mm above its waypoint while the IK reported a 0.26 mm
  residual. _WorldFrameProvider maps FK through the simulator's reported base
  pose, so the pose the policy is shown and the pose its IK solves in come from
  one code path in one frame.

Controller (measured, not guessed)

gz-sim's JointPositionController is a gz::math::PID; its law was read from the
gz-sim8 and gz-math7 sources and the accepted SDF parameters from the installed
library, not assumed. The world configured i_gain = 0 -- pure PD -- so a constant
gravity load left load/p_gain: 15.0 mrad on joint2, 17.9 on joint4, 31.5 on
joint7. The library's own i_max=-1/i_min=0 defaults leave iMax >= iMin false,
which DISABLES the integral clamp. With i_gain = 100 and i_max/i_min = +/-10 N,
the settled tool-error bound is 9.3 mm against the policy's own 20 mm reach
tolerance. cmd_max/cmd_min are set per joint from its effort limit, which
previously defaulted to no clamping at all.

The grasp is now contact (the latch is gone)

_update_grasp attached the object whenever the commanded aperture closed within
50 mm and ground_truth then reported the object at the end effector plus a
stored offset. No contact was resolved and no physics moved the object. It is
deleted: ground truth is the pose and orientation Gazebo wrote, and "grasped" is
derived from three measurements -- the aperture actually reached, the object's
measured position relative to the tool centre point, and its measured height
above the support surface. No code path writes the object's pose.

Measured outcome, seed 3, 0 mm, through run_episode

The arm reaches within 3.1 mm, the jaws enclose the object, and the object is
lifted 55.7 mm by contact alone and carried about 120 mm before leaving the
jaws. The episode reports FAIL and placement error is 0.125 m. No PASS is
claimed anywhere.

The 8 mm condition is NOT_SUPPORTED, not a failure: the camera noise really is
generated (stddev 0.008 m in the world) and the depth frame really is
delivered, but the object belief the policy receives is the simulator's pose --
the same convention simulation/mujoco.py uses -- so noise cannot reach the
policy. The run differs only because scenario_id participates in placement.
Reporting it as a noise failure would have been the exact error this project
exists to catch.

Evidence, tests, docs

scripts/gazebo_stage_check.py runs the Phase 3 ladder one stage at a time;
scripts/gazebo_pick_place_evidence.py records a real episode tick by tick.
22 new contract tests cover the boundary (readiness failure, joint-state
parsing, command mapping, reset isolation, shutdown, timeouts, observation
freshness, no mock fallback, frame coherence) and the measured geometry and
scene are pinned by further tests. docs/gazebo.md section 10 records every
defect as measurement -> cause -> change, with the commands to reproduce it.

pytest 521 passed / 8 skipped (baseline 497/8), ruff clean, mypy unchanged at
two pre-existing errors in the recording CLI.

File: gazebo/models/panda/panda.urdf (robot description, URDF)
Before this commit: robot panda, 11 links, 10 joints
Links:
- link panda_left_finger: geometry collision box size=0.02 0.015 0.017; visual box size=0.02 0.015 0.017
- link panda_right_finger: geometry collision box size=0.02 0.015 0.017; visual box size=0.02 0.015 0.017
Joints:
- joint left_finger: origin xyz=0 0 0.0584 rpy=0 0 0 -> xyz=0 0.0055 0.0445 rpy=0 0 0
- joint right_finger: origin xyz=0 -0.01 0.0584 rpy=0 0 0 -> xyz=0 -0.0055 0.0445 rpy=0 0 0

Commit message: Gazebo: a real pick and place, once -- and the contact system that made it possible
The previous commit ended with the grasp failing and inference from the object's
velocity standing in for evidence. Two things fixed: stop inferring, and load
the system that was missing.

The world had no contact system at all

In gz-sim8 the Collisions system no longer exists; collision pairs and
contact-sensor data come from gz::sim::systems::Contact, and the world loaded
Physics, UserCommands, SceneBroadcaster and Sensors without it. Loading it, and
putting contact sensors on the object and the table, changed the outcome of the
same episode from "never completes a carry" to "places the object 29.3 mm from
the target, inside the 50 mm tolerance".

Both pair sets now ride on Transition.info -- they are simulator facts, so they
are deliberately kept out of the Observation the policy reads -- and the evidence
run records them per tick. Nothing about the grip is inferred from how fast the
cube moved any more.

The pads were grazing the tabletop

The shared task aims the tool centre point at the object's centre, so the pad
lower edge lands at object_centre + pad_offset - pad_half_height. With an 8 mm
half-object on the table and an 8.5 mm pad, that is below the surface; the live
trace measured the arm settling 0.4 mm further low, so the lowest the pads ever
reached was +0.03 mm. Thirty microns is inside ODE's contact margin. MuJoCo
tolerates the same overlap -- the task's own feasibility test allows 1 mm --
which is why this never showed up before. The Gazebo pads are now 7.5 mm half
height, clearing the table by 1.03 mm and still spanning 15 mm of a 16 mm cube.
The test now pins the clearance rather than the raw height, because the clearance
is the quantity that matters and it is what the measurement was about.

Where it reaches, stated without inflation

One episode ran the task end to end: enclosed the object to 1.25 mm, held it for
26 ticks, lifted it 59.7 mm, carried it across the workspace and set it down
29.3 mm from the target. Every criterion passed except orientation, at 1.597 rad
against a 0.6 rad tolerance. For a cube the resting height cannot tell a yaw
from a tumble, so the evidence now records the object's quaternion.

That run is not reproducible. Four repeats of one configuration: one carried the
object, three lost it during or just after the lift (14.6, 0.0 and 0.0 mm). The
approach is deterministic and sub-millimetre; grasp retention is not. The
artifacts committed are from a failing repeat, deliberately -- a passing run I
cannot reproduce must not be presented as a result, and the JSON for the good run
was overwritten before it was saved.

The remaining problem is now narrow and stated: the pads reach the object, close
on it, and hold it for between 1 and 26 ticks depending on the run. That is a
grasp-retention problem with contact data available to attribute it, which is a
very different position from inferring the cause from the object's velocity.

The 8 mm condition stays NOT_SUPPORTED: the noise reaches the world but not the
policy, whose object belief is the simulator's pose.

pytest 523 passed / 8 skipped, ruff clean, mypy unchanged at two pre-existing
errors in the recording CLI.

File: gazebo/models/panda/panda.urdf (robot description, URDF)
Before this commit: robot panda, 11 links, 10 joints
Links:
- link panda_left_finger: geometry collision box size=0.02 0.015 0.015; visual box size=0.02 0.015 0.015
- link panda_right_finger: geometry collision box size=0.02 0.015 0.015; visual box size=0.02 0.015 0.015

Commit message: Gazebo: contact instrumentation, and the grasp blocker narrowed by elimination
Every claim about the Gazebo grasp so far was inferred from the object's
velocity: how fast it left the jaws, how far it was carried. That describes the
consequence, not the cause, and the two told different stories while the question
was open. This adds the measurement.

Contact sensors, and the failures that got them there

The world now loads gz::sim::systems::Contact and carries a contact sensor on
the object and on the table. Both pair sets ride on Transition.info, because
they are simulator facts and the Observation is what the policy may see.

Getting them to work took three wrong readings of the protobuf schema
(collisions[0], wrenches, wrench.force.normal), each of which raised inside the
callback so the subscriber reported no contacts at all while looking perfectly
healthy. The fix that mattered was not the third guess: the stream now counts
messages and keeps the first error, so a broken subscriber and a sensor with
nothing touching it can no longer look the same. It reports pair identity, the
one field verified against the running system; the per-body wrench magnitude is
left unread rather than guessed at a fourth time.

What the sensors say, over a full 149-tick episode

    cube    <-> table          149 ticks
    cube    <-> finger           0 ticks
    finger  <-> table          149 ticks

The jaws were closing on the tabletop and missing the object entirely. That also
explains the finger residual that survived every gain change: the pads were
pressed against the table and physically could not close.

The pads clear now, and the blocker is smaller but not gone

Shortening the pads to 6.5 mm half-height gives 2.0 mm of nominal clearance
against the arm's measured 1.4 mm sag, and table contact fell from every tick to
two. The cube is still never touched, and now the sensors prove the blocker is
not the table either: at the grasp the pads stall at a 21.4 mm separation on a
16 mm cube, with the tool 1.5 mm from the cube's centre and no contact anywhere.
A ~5 N per-pad command moving a 15 g finger at 0.0034 m/s needs a reaction and
the sensors report none, so it is neither the table, nor the cube, nor the pads
meeting each other. That is stated as an open question rather than a conclusion.

The squeeze-ejection hypothesis is recorded as overturned rather than deleted:
the pads were never in contact with the object, so nothing was being squeezed
out. Keeping a hypothesis that measurement refuted is worth as much as keeping
one it confirmed.

Unchanged: the episode still reports FAIL, 8 mm is still NOT_SUPPORTED, and the
paired comparison is still NOT_IMPLEMENTED. One run in this session did carry
the object 29.3 mm from the target with only the orientation criterion failing,
and it was not reproduced; the committed artifacts remain failing repeats.

pytest 523 passed / 8 skipped, ruff clean, mypy unchanged at two pre-existing
errors in the recording CLI.

File: gazebo/models/panda/panda.urdf (robot description, URDF)
Before this commit: robot panda, 11 links, 10 joints
Links:
- link panda_left_finger: geometry collision box size=0.02 0.015 0.013; visual box size=0.02 0.015 0.013
- link panda_right_finger: geometry collision box size=0.02 0.015 0.013; visual box size=0.02 0.015 0.013
